File: Hardware/ReflowControl.kicad_pcb (KiCad board)
At the start: 2 copper layers, 41.9 x 40.6 mm, 17 parts, among them J1 T Display RST Side, J2 T Display Empty Side, J3 T1, J4 T2, J5 T3, J6 I2C, J7 SSR, J8 Breakout

Commit message: Hard design update
Parts:
- R1: value 4.7k -> 1k
- R2: value 4.7k -> 2k
- R3: value 4.7k -> 5k
- moved J5 39.2 mm to (88.9, 123.2), turned to 180 degrees
- moved J7 35.7 mm to (88.9, 100.3), turned to 180 degrees
- moved C3 35.5 mm to (84.6, 124.8), turned to -90 degrees
- moved J8 35.1 mm to (48.3, 127.0), turned to -90 degrees
- moved J4 34.9 mm to (88.9, 115.6), turned to 180 degrees
- moved J3 33.6 mm to (88.9, 108.0), turned to 180 degrees
- moved R3 32.8 mm to (82.0, 124.7), turned to -90 degrees
- moved C1 29.8 mm to (84.6, 117.1), turned to -90 degrees
- moved R6 29.3 mm to (84.6, 101.6), turned to 90 degrees
- moved C2 27.5 mm to (84.6, 109.4), turned to -90 degrees
- moved R2 26.6 mm to (82.0, 117.1), turned to -90 degrees
- moved R1 23.9 mm to (82.0, 109.5), turned to -90 degrees
- moved J6 14.2 mm to (61.0, 105.4)
- moved R4 12.4 mm to (52.3, 104.1), turned to 0 degrees
- moved R5 4.97 mm to (52.3, 106.7), turned to 0 degrees
Connections:
- J1 pad 11: unconnected-(J1-Pin_11-Pad11) -> /THERM3
- J1 pad 7: unconnected-(J1-Pin_7-Pad7) -> /THERM2
- J1 pad 8: unconnected-(J1-Pin_8-Pad8) -> /THERM1
- J2 pad 7: /THERM3 -> unconnected-(J2-Pin_7-Pad7)
- J2 pad 8: /THERM2 -> unconnected-(J2-Pin_8-Pad8)
- J2 pad 9: /THERM1 -> unconnected-(J2-Pin_9-Pad9)
Routing:
- net /GPIO2: track 22.7 -> 60.9 mm
- net +5V: track 37.8 -> 5.08 mm
- net /THERM1: track 64.8 -> 33.9 mm
- net /GPIO27: track 35.8 -> 5.08 mm
- net /THERM3: track 52.2 -> 23.0 mm
- net +3.3V: track 106.0 -> 77.2 mm
- net /GPIO26: track 28.7 -> 5.08 mm
- net /GPIO25: track 27.5 -> 5.08 mm
- net GND: track 112.3 -> 132.0 mm
- net /GPIO33: track 22.4 -> 11.7 mm
- net /THERM2: track 57.5 -> 46.9 mm
- net /SCL: track 16.5 -> 22.9 mm
- net /SDA: track 17.4 -> 19.7 mm
Other:
- board size 41.9 x 40.6 mm -> 49.5 x 35.6 mm

Commit message: oopsie no2 - wrong board pin header orientation and added an s3 board as a secondary pin headout
Parts:
- added J10: S3-ZERO-SERIALSIDE, Connector_PinHeader_2.54mm:PinHeader_1x09_P2.54mm_Vertical, F.Cu at (68.6, 102.9)
- added J9: S3-ZERO-POWERSIDE, Connector_PinHeader_2.54mm:PinHeader_1x09_P2.54mm_Vertical, F.Cu at (48.3, 118.1)
- moved J2 27.9 mm to (76.2, 99.1), turned to -90 degrees
- moved J6 16.1 mm to (76.2, 110.5), turned to 90 degrees
- moved R4 8.13 mm to (58.7, 109.2)
- moved R5 8.13 mm to (58.7, 111.8)
Connections:
- net /GPIO25 renamed /GPIO25_8
- net /GPIO26 renamed /GPIO26_7
- net /GPIO27 renamed /GPIO27_RX
- net /GPIO33 renamed /GPIO33_TX
Routing:
- net /GPIO26_7: track 5.08 -> 79.6 mm
- net /GPIO25_8: track 5.08 -> 76.4 mm
- net /THERM1: track 33.9 -> 86.6 mm
- net /THERM3: track 23.0 -> 56.1 mm
- net /GPIO33_TX: track 11.7 -> 39.3 mm
- net /GPIO27_RX: track 5.08 -> 32.3 mm
- net +3.3V: track 77.2 -> 103.5 mm
- net /THERM2: track 46.9 -> 71.2 mm
- net /SDA: track 19.7 -> 33.3 mm
- net GND: track 132.0 -> 143.6 mm
- net /SCL: track 22.9 -> 29.9 mm
- net +5V: track 5.08 -> 8.89 mm
- net /GPIO2: track 60.9 -> 63.8 mm
