File: Hardware/ReflowControl.kicad_sch (KiCad schematic)
At the start: 17 parts, among them J1 T Display RST Side, J2 T Display Empty Side, J3 T1, J4 T2, J5 T3, J6 I2C, J7 SSR, J8 Breakout

Commit message: Hard design update
Parts:
- R1: value 4.7k -> 1k
- R2: value 4.7k -> 2k
- R3: value 4.7k -> 5k
Connections:
- net THERM1: now also J1.8 (Pin_8); no longer J2.9 (Pin_9)
- net THERM2: now also J1.7 (Pin_7); no longer J2.8 (Pin_8)
- net THERM3: now also J1.11 (Pin_11); no longer J2.7 (Pin_7)
Changed lines of the file:
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@@
 	(wire
 		(pts
-			(xy 135.89 97.79) (xy 142.24 97.79)
+			(xy 90.17 57.15) (xy 100.33 57.15)
 		)
 		(stroke
@@
 	(wire
 		(pts
-			(xy 71.12 93.98) (xy 71.12 99.06)
+			(xy 135.89 97.79) (xy 142.24 97.79)
 		)
 		(stroke
@@
 	(wire
 		(pts
-			(xy 71.12 24.13) (xy 71.12 26.67)
+			(xy 71.12 93.98) (xy 71.12 99.06)
 		)
 		(stroke
@@
 	(wire
 		(pts
-			(xy 62.23 125.73) (xy 85.09 125.73)
+			(xy 71.12 24.13) (xy 71.12 26.67)
 		)
 		(stroke
@@
 	(wire
 		(pts
-			(xy 54.61 80.01) (xy 54.61 77.47)
+			(xy 62.23 125.73) (xy 85.09 125.73)
 		)
 		(stroke
@@
 	(wire
 		(pts
-			(xy 85.09 135.89) (xy 52.07 135.89)
+			(xy 54.61 80.01) (xy 54.61 77.47)
 		)
 		(stroke
@@
 	(wire
 		(pts
-			(xy 62.23 111.76) (xy 62.23 116.84)
+			(xy 85.09 135.89) (xy 52.07 135.89)
 		)
 		(stroke
@@
 	(wire
 		(pts
-			(xy 50.8 72.39) (xy 57.15 72.39)
+			(xy 62.23 111.76) (xy 62.23 116.84)
 		)
 		(stroke
@@
 	(wire
 		(pts
-			(xy 50.8 69.85) (xy 57.15 69.85)
+			(xy 90.17 67.31) (xy 100.33 67.31)
 		)
 		(stroke
@@
 	(wire
 		(pts
+			(xy 90.17 54.61) (xy 109.22 54.61)
+		)
+		(stroke
+			(width 0)
+			(type default)
+		)
+	)
+	(wire
+		(pts
 			(xy 48.26 111.76) (xy 62.23 111.76)
 		)
@@
 	(wire
 		(pts
-			(xy 71.12 24.13) (xy 67.31 24.13)
+			(xy 90.17 64.77) (xy 100.33 64.77)
 		)
 		(stroke
@@
 	(wire
 		(pts
-			(xy 48.26 138.43) (xy 62.23 138.43)
+			(xy 71.12 24.13) (xy 67.31 24.13)
 		)
 		(stroke
@@
 	(wire
 		(pts
-			(xy 90.17 54.61) (xy 100.33 54.61)
+			(xy 48.26 138.43) (xy 62.23 138.43)
 		)
 		(stroke
@@
 	(wire
 		(pts
-			(xy 50.8 74.93) (xy 57.15 74.93)
-		)
-		(stroke
-			(width 0)
-			(type default)
-		)
-	)
-	(wire
-		(pts
 			(xy 135.89 102.87) (xy 142.24 102.87)
 		)
@@
 	)
 	(label "THERM1"
-		(at 50.8 74.93 180)
+		(at 100.33 64.77 0)
 		(fields_autoplaced yes)
 		(effects
@@
 				(size 1.27 1.27)
 			)
-			(justify right bottom)
+			(justify left bottom)
 		)
 	)
 	(label "THERM2"
-		(at 50.8 72.39 180)
+		(at 100.33 67.31 0)
 		(fields_autoplaced yes)
 		(effects
@@
 				(size 1.27 1.27)
 			)
-			(justify right bottom)
+			(justify left bottom)
 		)
 	)
@@
 	)
 	(label "THERM3"
-		(at 50.8 69.85 180)
+		(at 100.33 57.15 0)
 		(fields_autoplaced yes)
 		(effects
@@
 				(size 1.27 1.27)
 			)
-			(justify right bottom)
+			(justify left bottom)
 		)
 	)
@@
 			)
 		)
-		(property "Value" "4.7k"
+		(property "Value" "5k"
 			(at 68.58 140.97 90)
 			(effects
@@
 			)
 		)
-		(property "Value" "4.7k"
+		(property "Value" "1k"
 			(at 68.58 114.3 90)
 			(effects
@@
 	(symbol
 		(lib_id "power:+3.3V")
-		(at 100.33 54.61 270)
+		(at 109.22 54.61 270)
 		(unit 1)
 		(exclude_from_sim no)
@@
 		(dnp no)
 		(property "Reference" "#PWR04"
-			(at 96.52 54.61 0)
+			(at 105.41 54.61 0)
 			(effects
 				(font
@@
 		)
 		(property "Value" "+3.3V"
-			(at 103.378 54.61 90)
+			(at 112.268 54.61 90)
 			(effects
 				(font
@@
 		)
 		(property "Footprint" ""
-			(at 100.33 54.61 0)
+			(at 109.22 54.61 0)
 			(effects
 				(font
@@
 		)
 		(property "Datasheet" ""
-			(at 100.33 54.61 0)
+			(at 109.22 54.61 0)
 			(effects
 				(font
@@
 		)
 		(property "Description" "Power symbol creates a global label with name \"+3.3V\""
-			(at 100.33 54.61 0)
+			(at 109.22 54.61 0)
 			(effects
 				(font
@@
 			)
 		)
-		(property "Value" "4.7k"
+		(property "Value" "2k"
 			(at 68.58 128.27 90)
 			(effects

Commit message: oopsie no2 - wrong board pin header orientation and added an s3 board as a secondary pin headout
Parts:
- added J10: S3-ZERO-SERIALSIDE, Connector_PinHeader_2.54mm:PinHeader_1x09_P2.54mm_Vertical, symbol Connector_Generic:Conn_01x09
- added J9: S3-ZERO-POWERSIDE, Connector_PinHeader_2.54mm:PinHeader_1x09_P2.54mm_Vertical, symbol Connector_Generic:Conn_01x09
Connections:
- net +3.3V: now also J9.3 (Pin_3)
- net +5V: now also J9.1 (Pin_1)
- net GND: now also J9.2 (Pin_2)
- net GPIO2: now also J9.5 (Pin_5)
- net SCL: now also J9.9 (Pin_9)
- net SDA: now also J9.8 (Pin_8)
- net THERM1: now also J10.7 (Pin_7)
- net THERM2: now also J10.6 (Pin_6)
- net THERM3: now also J10.5 (Pin_5)
- net GPIO25 renamed GPIO25_8
- net GPIO25_8: now also J10.2 (Pin_2)
- net GPIO26 renamed GPIO26_7
- net GPIO26_7: now also J10.1 (Pin_1)
- net GPIO27 renamed GPIO27_RX
- net GPIO27_RX: now also J10.8 (Pin_8)
- net GPIO33 renamed GPIO33_TX
- net GPIO33_TX: now also J10.9 (Pin_9)
- new net GPIO1: J9.4 (Pin_4)
- new net GPIO10: J10.4 (Pin_4)
- new net GPIO3: J9.6 (Pin_6)
- new net GPIO4: J9.7 (Pin_7)
- new net GPIO9: J10.3 (Pin_3)
Other:
- note added: "GPIO33_TX - On the t-display, this is GPIO33, on the S3 its TX GPIO27_RX - On the t-display, this is GPIO24, on the S3 its RX GPIO25_8 - On the t-display, this is GPIO25, on the S3 its 8 GPIO26_7 - On the t-display, this is GPIO26, on the S3 its 7"
